File: hardware/AIC8800M/FEM_5G.kicad_sch (KiCad schematic)
At the start: 25 parts, among them U4 CB5717/SKY85717-21

Commit message: [hardware/AIC8800m] update [vsf] sync
Connections:
- no-connect marks 1 -> 0
Changed lines of the file:
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@@
   (junction (at 163.83 107.95) (diameter 0) (color 0 0 0 0)
   )
-  (no_connect (at -22.86 107.95))
   (wire (pts (xy 172.72 58.42) (xy 173.99 58.42))
     (stroke (width 0) (type default))
@@
     (pin "2")
     (instances
-      (project "aic8800m_basic"
+      (project "MCULinux"
         (path "/b0717bb8-5e5d-44de-b48f-ff278896fb50/00000000-0000-0000-0000-000061f4753e"
           (reference "AE3") (unit 1)
@@
     (pin "1")
     (instances
-      (project "aic8800m_basic"
+      (project "MCULinux"
         (path "/b0717bb8-5e5d-44de-b48f-ff278896fb50/00000000-0000-0000-0000-000061f4753e"
           (reference "#PWR055") (unit 1)
@@
     (pin "2")
     (instances
-      (project "aic8800m_basic"
+      (project "MCULinux"
         (path "/b0717bb8-5e5d-44de-b48f-ff278896fb50/00000000-0000-0000-0000-000061f4753e"
           (reference "L10") (unit 1)
@@
     (pin "2")
     (instances
-      (project "aic8800m_basic"
+      (project "MCULinux"
         (path "/b0717bb8-5e5d-44de-b48f-ff278896fb50/00000000-0000-0000-0000-000061f4753e"
           (reference "C50") (unit 1)
@@
     (pin "2")
     (instances
-      (project "aic8800m_basic"
+      (project "MCULinux"
         (path "/b0717bb8-5e5d-44de-b48f-ff278896fb50/00000000-0000-0000-0000-000061f4753e"
           (reference "C54") (unit 1)
@@
     (pin "1")
     (instances
-      (project "aic8800m_basic"
+      (project "MCULinux"
         (path "/b0717bb8-5e5d-44de-b48f-ff278896fb50/00000000-0000-0000-0000-000061f4753e"
           (reference "#PWR051") (unit 1)
@@
     (pin "1")
     (instances
-      (project "aic8800m_basic"
+      (project "MCULinux"
         (path "/b0717bb8-5e5d-44de-b48f-ff278896fb50/00000000-0000-0000-0000-000061f4753e"
           (reference "#PWR056") (unit 1)
@@
     (pin "2")
     (instances
-      (project "aic8800m_basic"
+      (project "MCULinux"
         (path "/b0717bb8-5e5d-44de-b48f-ff278896fb50/00000000-0000-0000-0000-000061f4753e"
           (reference "L9") (unit 1)
@@
     (pin "1")
     (instances
-      (project "aic8800m_basic"
+      (project "MCULinux"
         (path "/b0717bb8-5e5d-44de-b48f-ff278896fb50/00000000-0000-0000-0000-000061f4753e"
           (reference "#PWR052") (unit 1)
@@
     (pin "1")
     (instances
-      (project "aic8800m_basic"
+      (project "MCULinux"
         (path "/b0717bb8-5e5d-44de-b48f-ff278896fb50/00000000-0000-0000-0000-000061f4753e"
           (reference "#PWR049") (unit 1)
@@
     (pin "2")
     (instances
-      (project "aic8800m_basic"
+      (project "MCULinux"
         (path "/b0717bb8-5e5d-44de-b48f-ff278896fb50/00000000-0000-0000-0000-000061f4753e"
           (reference "C52") (unit 1)
@@
     (pin "2")
     (instances
-      (project "aic8800m_basic"
+      (project "MCULinux"
         (path "/b0717bb8-5e5d-44de-b48f-ff278896fb50/00000000-0000-0000-0000-000061f4753e"
           (reference "C48") (unit 1)
@@
     (pin "2")
     (instances
-      (project "aic8800m_basic"
+      (project "MCULinux"
         (path "/b0717bb8-5e5d-44de-b48f-ff278896fb50/00000000-0000-0000-0000-000061f4753e"
           (reference "R34") (unit 1)
@@
     (pin "2")
     (instances
-      (project "aic8800m_basic"
+      (project "MCULinux"
         (path "/b0717bb8-5e5d-44de-b48f-ff278896fb50/00000000-0000-0000-0000-000061f4753e"
           (reference "C46") (unit 1)
@@
     (pin "1")
     (instances
-      (project "aic8800m_basic"
+      (project "MCULinux"
         (path "/b0717bb8-5e5d-44de-b48f-ff278896fb50/00000000-0000-0000-0000-000061f4753e"
           (reference "#PWR047") (unit 1)
@@
     (pin "2")
     (instances
-      (project "aic8800m_basic"
+      (project "MCULinux"
         (path "/b0717bb8-5e5d-44de-b48f-ff278896fb50/00000000-0000-0000-0000-000061f4753e"
           (reference "C47") (unit 1)
@@
     (pin "1")
     (instances
-      (project "aic8800m_basic"
+      (project "MCULinux"
         (path "/b0717bb8-5e5d-44de-b48f-ff278896fb50/00000000-0000-0000-0000-000061f4753e"
           (reference "#PWR048") (unit 1)
@@
     (pin "2")
     (instances
-      (project "aic8800m_basic"
+      (project "MCULinux"
         (path "/b0717bb8-5e5d-44de-b48f-ff278896fb50/00000000-0000-0000-0000-000061f4753e"
           (reference "C51") (unit 1)
@@
     (pin "2")
     (instances
-      (project "aic8800m_basic"
+      (project "MCULinux"
         (path "/b0717bb8-5e5d-44de-b48f-ff278896fb50/00000000-0000-0000-0000-000061f4753e"
           (reference "C49") (unit 1)
@@
     (pin "1")
     (instances
-      (project "aic8800m_basic"
+      (project "MCULinux"
         (path "/b0717bb8-5e5d-44de-b48f-ff278896fb50/00000000-0000-0000-0000-000061f4753e"
           (reference "#PWR053") (unit 1)
@@
     (pin "1")
     (instances
-      (project "aic8800m_basic"
+      (project "MCULinux"
         (path "/b0717bb8-5e5d-44de-b48f-ff278896fb50/00000000-0000-0000-0000-000061f4753e"
           (reference "#PWR050") (unit 1)
@@
     (pin "2")
     (instances
-      (project "aic8800m_basic"
+      (project "MCULinux"
         (path "/b0717bb8-5e5d-44de-b48f-ff278896fb50/00000000-0000-0000-0000-000061f4753e"
           (reference "C43") (unit 1)
@@
     (pin "1")
     (instances
-      (project "aic8800m_basic"
+      (project "MCULinux"
         (path "/b0717bb8-5e5d-44de-b48f-ff278896fb50/00000000-0000-0000-0000-000061f4753e"
           (reference "#PWR042") (unit 1)
@@
     (pin "1")
     (instances
-      (project "aic8800m_basic"
+      (project "MCULinux"
         (path "/b0717bb8-5e5d-44de-b48f-ff278896fb50/00000000-0000-0000-0000-000061f4753e"
           (reference "#PWR044") (unit 1)
@@
     (pin "2")
     (instances
-      (project "aic8800m_basic"
+      (project "MCULinux"
         (path "/b0717bb8-5e5d-44de-b48f-ff278896fb50/00000000-0000-0000-0000-000061f4753e"
           (reference "C45") (unit 1)
@@
     (pin "1")
     (instances
-      (project "aic8800m_basic"
+      (project "MCULinux"
         (path "/b0717bb8-5e5d-44de-b48f-ff278896fb50/00000000-0000-0000-0000-000061f4753e"
           (reference "#PWR046") (unit 1)
@@
     (pin "2")
     (instances
-      (project "aic8800m_basic"
+      (project "MCULinux"
         (path "/b0717bb8-5e5d-44de-b48f-ff278896fb50/00000000-0000-0000-0000-000061f4753e"
           (reference "C41") (unit 1)
@@
     (pin "2")
     (instances
-      (project "aic8800m_basic"
+      (project "MCULinux"
         (path "/b0717bb8-5e5d-44de-b48f-ff278896fb50/00000000-0000-0000-0000-000061f4753e"
           (reference "L8") (unit 1)
@@
     (pin "2")
     (instances
-      (project "aic8800m_basic"
+      (project "MCULinux"
         (path "/b0717bb8-5e5d-44de-b48f-ff278896fb50/00000000-0000-0000-0000-000061f4753e"
           (reference "C40") (unit 1)
@@
     (pin "1")
     (instances
-      (project "aic8800m_basic"
+      (project "MCULinux"
         (path "/b0717bb8-5e5d-44de-b48f-ff278896fb50/00000000-0000-0000-0000-000061f4753e"
           (reference "#PWR041") (unit 1)
@@
     (pin "2")
     (instances
-      (project "aic8800m_basic"
+      (project "MCULinux"
         (path "/b0717bb8-5e5d-44de-b48f-ff278896fb50/00000000-0000-0000-0000-000061f4753e"
           (reference "C42") (unit 1)
@@
     (pin "1")
     (instances
-      (project "aic8800m_basic"
+      (project "MCULinux"
         (path "/b0717bb8-5e5d-44de-b48f-ff278896fb50/00000000-0000-0000-0000-000061f4753e"
           (reference "#PWR043") (unit 1)
@@
     (pin "1")
     (instances
-      (project "aic8800m_basic"
+      (project "MCULinux"
         (path "/b0717bb8-5e5d-44de-b48f-ff278896fb50/00000000-0000-0000-0000-000061f4753e"
           (reference "#PWR045") (unit 1)
@@
     (pin "2")
     (instances
-      (project "aic8800m_basic"
+      (project "MCULinux"
         (path "/b0717bb8-5e5d-44de-b48f-ff278896fb50/00000000-0000-0000-0000-000061f4753e"
           (reference "C44") (unit 1)
@@
     (pin "1")
     (instances
-      (project "aic8800m_basic"
+      (project "MCULinux"
         (path "/b0717bb8-5e5d-44de-b48f-ff278896fb50/00000000-0000-0000-0000-000061f4753e"
           (reference "#PWR054") (unit 1)
@@
     (pin "2")
     (instances
-      (project "aic8800m_basic"
+      (project "MCULinux"
         (path "/b0717bb8-5e5d-44de-b48f-ff278896fb50/00000000-0000-0000-0000-000061f4753e"
           (reference "C53") (unit 1)
@@
     (pin "1")
     (instances
-      (project "aic8800m_basic"
+      (project "MCULinux"
         (path "/b0717bb8-5e5d-44de-b48f-ff278896fb50/00000000-0000-0000-0000-000061f4753e"
           (reference "#PWR057") (unit 1)
@@
     (pin "2")
     (instances
-      (project "aic8800m_basic"
+      (project "MCULinux"
         (path "/b0717bb8-5e5d-44de-b48f-ff278896fb50/00000000-0000-0000-0000-000061f4753e"
           (reference "C55") (unit 1)
@@
     (pin "2")
     (instances
-      (project "aic8800m_basic"
+      (project "MCULinux"
         (path "/b0717bb8-5e5d-44de-b48f-ff278896fb50/00000000-0000-0000-0000-000061f4753e"
           (reference "R31") (unit 1)
@@
     (pin "2")
     (instances
-      (project "aic8800m_basic"
+      (project "MCULinux"
         (path "/b0717bb8-5e5d-44de-b48f-ff278896fb50/00000000-0000-0000-0000-000061f4753e"
           (reference "R33") (unit 1)
@@
     (pin "2")
     (instances
-      (project "aic8800m_basic"
+      (project "MCULinux"
         (path "/b0717bb8-5e5d-44de-b48f-ff278896fb50/00000000-0000-0000-0000-000061f4753e"
           (reference "R32") (unit 1)
@@
     (pin "9")
     (instances
-      (project "aic8800m_basic"
+      (project "MCULinux"
         (path "/b0717bb8-5e5d-44de-b48f-ff278896fb50/00000000-0000-0000-0000-000061f4753e"
           (reference "U4") (unit 1)
