File: hardware/AIC8800M/MCULinux.kicad_sch (KiCad schematic)
At the start: 75 parts, among them J1 USB_C_Receptacle_USB2.0, J2 USB_C_Receptacle_USB2.0, J3 USB_A, Q1 S9013, SW1 SW_Push, SW2 SW_Push, SW3 SW_Push, SW4 SW_Push, U1 AIC8800M_48P, U2 CH340N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

Commit message: [hardware/AIC8800m] update [vsf] sync
Parts:
- added R13 (x2): 1k, Resistor_SMD:R_0402_1005Metric, symbol Device:R
- C3, C4: footprint Capacitor_SMD:C_0603_1608Metric -> Capacitor_SMD:C_0402_1005Metric
- C5: footprint Capacitor_SMD:C_0805_2012Metric -> Capacitor_SMD:C_0402_1005Metric
- D3, D5, D6: footprint Diode_THT:D_DO-35_SOD27_P7.62mm_Horizontal -> Diode_SMD:D_SOD-123F
- Q1: footprint (none) -> Package_TO_SOT_SMD:SOT-23
Connections:
- net LCD_CS is gone; now on net GPIOA11: J4.13 (CS)
- net LCD_MOSI is gone; now on net GPIOA13: J4.11 (SDA)
- net LCD_RS is gone; now on net GPIOA12: J4.12 (RS)
- net LCD_SCK is gone; now on net GPIOA10: J4.9 (SCL)
- net TP_RST is gone; now on net LCD_RST: J4.16 (TP_RESET)
- net TP_SCL is gone; now on net GPIOA14: J4.19 (TP_SCL)
- net TP_SDA is gone; now on net GPIOA15: J4.18 (TP_SDA)
- net UART_RX is gone; now on net GPIOA8: U2.6 (TXD)
- net UART_TX is gone; now on net GPIOA9: U2.7 (RXD)
- net GND: now also R13.2
- net VBAT: now also R13.2
- new net: R13.1, R13.1
- no-connect marks 1 -> 0
Other:
- moved on the sheet: D3, D5, D6, J4, Q1, R13, R9
